File: clock/clock.kicad_sch (KiCad schematic)
At the start: 88 parts, among them J1 Power_inlet_vertical, J2 Conn_01x06, J3 Conn_02x03_Odd_Even, SW1 Omron_B3F_SPST, SW2 Omron_B3F_SPST, SW3 Omron_B3F_SPST, SW4 Omron_B3F_SPST, SW5 Omron_B3F_SPST, U1 ATmega328-PU, U2 L7805, U3 MAX7219, U4 DS1307_DIP-8, U5 UltrasonicModule, Y1 16MHz, Y2 Crystal_32768Hz

Commit message: update
Connections:
- net VCC: now also D10.3 (VDD)
- no-connect marks 7 -> 10
Changed lines of the file:
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@@
   (junction (at 39.37 243.84) (diameter 0) (color 0 0 0 0)
   )
+  (no_connect (at 66.04 76.2))
+  (no_connect (at 66.04 73.66))
   (no_connect (at 57.15 201.93))
   (no_connect (at 57.15 199.39))
   (no_connect (at 57.15 204.47))
+  (no_connect (at 386.08 207.01))
   (no_connect (at 175.26 90.17))
   (no_connect (at 199.39 44.45))
@@
     (stroke (width 0) (type default) (color 0 0 0 0))
   )
-  (wire (pts (xy 288.29 153.67) (xy 294.64 153.67))
-    (stroke (width 0) (type default) (color 0 0 0 0))
-  )
   (wire (pts (xy 350.52 187.96) (xy 350.52 195.58))
     (stroke (width 0) (type default) (color 0 0 0 0))
@@
     (stroke (width 0) (type default) (color 0 0 0 0))
   )
+  (wire (pts (xy 288.29 153.67) (xy 294.64 153.67))
+    (stroke (width 0) (type default) (color 0 0 0 0))
+  )
   (wire (pts (xy 44.45 209.55) (xy 44.45 212.09))
     (stroke (width 0) (type default) (color 0 0 0 0))
@@
     (pin "1")
   )
-  (symbol (lib_id "HPS:VCC") (at 274.955 203.835 90) (unit 1)
+  (symbol (lib_id "HPS:VCC") (at 272.415 201.295 270) (unit 1)
     (in_bom yes) (on_board yes) (fields_autoplaced)
-    (property "Reference" "#PWR0160" (id 0) (at 278.765 203.835 0)
+    (property "Reference" "#PWR0160" (id 0) (at 268.605 201.295 0)
       (effects (font (size 1.27 1.27)) hide)
     )
-    (property "Value" "VCC" (id 1) (at 276.225 203.1999 90)
-      (effects (font (size 1.27 1.27)) (justify right))
+    (property "Value" "VCC" (id 1) (at 276.86 203.1999 90)
+      (effects (font (size 1.27 1.27)) (justify left))
     )
-    (property "Footprint" "" (id 2) (at 274.955 203.835 0)
+    (property "Footprint" "" (id 2) (at 272.415 201.295 0)
       (effects (font (size 1.27 1.27)) hide)
     )
-    (property "Datasheet" "" (id 3) (at 274.955 203.835 0)
+    (property "Datasheet" "" (id 3) (at 272.415 201.295 0)
       (effects (font (size 1.27 1.27)) hide)
     )
@@
     (pin "1")
   )
+  (symbol (lib_id "HPS:GND") (at 288.29 154.94 0) (unit 1)
+    (in_bom yes) (on_board yes) (fields_autoplaced)
+    (property "Reference" "#PWR0207" (id 0) (at 288.29 161.29 0)
+      (effects (font (size 1.27 1.27)) hide)
+    )
+    (property "Value" "GND" (id 1) (at 287.02 158.75 0))
+    (property "Footprint" "" (id 2) (at 288.29 154.94 0)
+      (effects (font (size 1.27 1.27)) hide)
+    )
+    (property "Datasheet" "" (id 3) (at 288.29 154.94 0)
+      (effects (font (size 1.27 1.27)) hide)
+    )
+    (pin "1")
+  )
   (symbol (lib_id "HPS:GND") (at 171.45 96.52 0) (unit 1)
     (in_bom yes) (on_board yes)
@@
     (pin "2")
   )
-  (symbol (lib_id "HPS:GND") (at 288.29 154.94 0) (unit 1)
-    (in_bom yes) (on_board yes) (fields_autoplaced)
-    (property "Reference" "#PWR0207" (id 0) (at 288.29 161.29 0)
-      (effects (font (size 1.27 1.27)) hide)
-    )
-    (property "Value" "GND" (id 1) (at 287.02 158.75 0))
-    (property "Footprint" "" (id 2) (at 288.29 154.94 0)
-      (effects (font (size 1.27 1.27)) hide)
-    )
-    (property "Datasheet" "" (id 3) (at 288.29 154.94 0)
-      (effects (font (size 1.27 1.27)) hide)
-    )
-    (pin "1")
-  )
   (symbol (lib_id "HPS:GND") (at 288.29 58.42 0) (unit 1)
     (in_bom yes) (on_board yes) (fields_autoplaced)
@@
       (reference "#PWR0206") (unit 1) (value "VCC") (footprint "")
     )
-    (path "/f3c0e85a-0dda-4cd6-acb7-34e5a38afe1e"
+    (path "/da5292c1-7475-48bc-a037-e772a8e51c7e"
       (reference "#PWR0207") (unit 1) (value "GND") (footprint "")
     )
