File: clock/clock.kicad_pcb (KiCad board)
At the start: 2 copper layers, 118 x 118 mm, 122 parts, among them J1 PJ-102AH, J2 Conn_01x06, J3 Conn_02x03_Odd_Even, SW1 Omron_B3F_SPST, SW2 Omron_B3F_SPST, SW3 Omron_B3F_SPST, SW4 Omron_B3F_SPST, SW5 Omron_B3F_SPST, U1 ATmega328-PU, U3 MAX7219, U4 DS1307_DIP-8, Y1 16MHz, Y2 Crystal_32768Hz

Commit message: update
Parts:
- removed C14, C15, C16, C17, C18, C19, C20, C21, C22, C23, C24, C25, C26, C27, C28, C29, C30, C31, C32, C33, C34, C35, C36, C37, C38, C39, C40, C41, C42, C43, C44, C45, C46, C47, C48, C49: 0.1uf, footprints:C_0805_2012Metric
- removed the H1 at (150.0, 45.5)
- removed the H2 at (204.5, 100.0)
- removed the H3 at (150.0, 154.5)
- removed the H4 at (95.5, 100.0)
- added H1 (x2): MountingHole, footprints:MountingHole_3.2mm_M3, F.Cu at (84.9, 56.2)
- added H2 (x2): MountingHole, footprints:MountingHole_3.2mm_M3, F.Cu at (214.9, 56.2)
- added H3: MountingHole, footprints:MountingHole_3.2mm_M3, F.Cu at (129.5, 10.2)
- added H3: MountingHole, footprints:MountingHole_3.2mm_M3, F.Cu at (84.9, 136.2)
- added H4 (x2): MountingHole, footprints:MountingHole_3.2mm_M3, F.Cu at (214.9, 136.2)
- added U2: L7805, footprints:TO-252-2, F.Cu at (200.7, 103.7)
- added U5: UltrasonicModule, footprints:HC-SR04_Horiz, F.Cu at (148.1, 68.6)
- C10, C11, C12, C13: value 0.1uf -> 10uf
- moved D10 391.1 mm to (104.0, 256.5)
- moved D9 375.6 mm to (104.0, 246.4)
- moved D20 364.5 mm to (119.3, 256.5)
- moved D7 364.2 mm to (104.0, 226.1)
- moved D27 357.7 mm to (132.0, 226.1)
- moved D38 341.5 mm to (144.7, 236.2)
- moved D17 330.8 mm to (119.4, 227.0)
- moved D19 330.1 mm to (119.3, 246.4)
- moved D3 323.3 mm to (104.0, 186.4)
- moved D37 322.0 mm to (144.7, 226.1)
- moved D14 320.0 mm to (119.3, 195.6)
- moved D1 318.8 mm to (104.0, 168.6)
- moved D13 318.8 mm to (119.3, 186.4)
- moved D25 318.6 mm to (132.0, 205.7)
- moved D30 314.5 mm to (132.0, 256.5)
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Connections:
- C10 pad 1: Net-(C10-Pad1) -> VCC
- C10 pad 2: VCC -> GND
- C11 pad 1: Net-(C11-Pad1) -> VCC
- C11 pad 2: VCC -> GND
- C12 pad 1: Net-(C12-Pad1) -> VCC
- C12 pad 2: VCC -> GND
- C13 pad 1: Net-(C13-Pad1) -> VCC
- C13 pad 2: VCC -> GND
- D1 pad 3: Net-(C10-Pad1) -> VCC
- D10 pad 3: Net-(C19-Pad1) -> VCC
- D11 pad 2: Net-(D11-Pad2) -> Net-(D10-Pad4)
- D11 pad 3: Net-(C29-Pad1) -> VCC
- D12 pad 2: Net-(D12-Pad2) -> Net-(D11-Pad4)
- D12 pad 3: Net-(C28-Pad1) -> VCC
- D12 pad 4: Net-(D11-Pad2) -> Net-(D12-Pad4)
- D13 pad 2: Net-(D13-Pad2) -> Net-(D12-Pad4)
- D13 pad 3: Net-(C27-Pad1) -> VCC
- D13 pad 4: Net-(D12-Pad2) -> Net-(D13-Pad4)
- D14 pad 2: Net-(D14-Pad2) -> Net-(D13-Pad4)
- D14 pad 3: Net-(C26-Pad1) -> VCC
- D14 pad 4: Net-(D13-Pad2) -> Net-(D14-Pad4)
- D15 pad 2: Net-(D15-Pad2) -> Net-(D14-Pad4)
- D15 pad 3: Net-(C25-Pad1) -> VCC
- D15 pad 4: Net-(D14-Pad2) -> Net-(D15-Pad4)
- D16 pad 2: Net-(D16-Pad2) -> Net-(D15-Pad4)
- D16 pad 3: Net-(C24-Pad1) -> VCC
- D16 pad 4: Net-(D15-Pad2) -> Net-(D16-Pad4)
- D17 pad 2: Net-(D17-Pad2) -> Net-(D16-Pad4)
- D17 pad 3: Net-(C23-Pad1) -> VCC
- D17 pad 4: Net-(D16-Pad2) -> Net-(D17-Pad4)
- D18 pad 2: Net-(D18-Pad2) -> Net-(D17-Pad4)
- D18 pad 3: Net-(C22-Pad1) -> VCC
- D18 pad 4: Net-(D17-Pad2) -> Net-(D18-Pad4)
- D19 pad 2: Net-(D19-Pad2) -> Net-(D18-Pad4)
- D19 pad 3: Net-(C21-Pad1) -> VCC
- D19 pad 4: Net-(D18-Pad2) -> Net-(D19-Pad4)
- D2 pad 3: Net-(C11-Pad1) -> VCC
- D20 pad 2: Net-(D10-Pad4) -> Net-(D19-Pad4)
- D20 pad 3: Net-(C20-Pad1) -> VCC
- D20 pad 4: Net-(D19-Pad2) -> Net-(D20-Pad4)
- D21 pad 2: Net-(D11-Pad4) -> Net-(D20-Pad4)
- D21 pad 3: Net-(C30-Pad1) -> VCC
- D22 pad 3: Net-(C31-Pad1) -> VCC
- D23 pad 3: Net-(C32-Pad1) -> VCC
- D24 pad 3: Net-(C33-Pad1) -> VCC
- D25 pad 3: Net-(C34-Pad1) -> VCC
- D26 pad 3: Net-(C35-Pad1) -> VCC
- D27 pad 3: Net-(C36-Pad1) -> VCC
- D28 pad 3: Net-(C37-Pad1) -> VCC
- D29 pad 3: Net-(C38-Pad1) -> VCC
- D3 pad 3: Net-(C12-Pad1) -> VCC
- D30 pad 3: Net-(C39-Pad1) -> VCC
- D31 pad 2: Net-(D31-Pad2) -> Net-(D30-Pad4)
- D31 pad 3: Net-(C49-Pad1) -> VCC
- D31 pad 4: unconnected-(D31-Pad4) -> Net-(D31-Pad4)
- D32 pad 2: Net-(D32-Pad2) -> Net-(D31-Pad4)
- D32 pad 3: Net-(C48-Pad1) -> VCC
- D32 pad 4: Net-(D31-Pad2) -> Net-(D32-Pad4)
- D33 pad 2: Net-(D33-Pad2) -> Net-(D32-Pad4)
- D33 pad 3: Net-(C47-Pad1) -> VCC
- D33 pad 4: Net-(D32-Pad2) -> Net-(D33-Pad4)
- D34 pad 2: Net-(D34-Pad2) -> Net-(D33-Pad4)
- D34 pad 3: Net-(C46-Pad1) -> VCC
- D34 pad 4: Net-(D33-Pad2) -> Net-(D34-Pad4)
- D35 pad 2: Net-(D35-Pad2) -> Net-(D34-Pad4)
- D35 pad 3: Net-(C45-Pad1) -> VCC
- D35 pad 4: Net-(D34-Pad2) -> Net-(D35-Pad4)
- D36 pad 2: Net-(D36-Pad2) -> Net-(D35-Pad4)
- D36 pad 3: Net-(C44-Pad1) -> VCC
- D36 pad 4: Net-(D35-Pad2) -> Net-(D36-Pad4)
- D37 pad 2: Net-(D37-Pad2) -> Net-(D36-Pad4)
- D37 pad 3: Net-(C43-Pad1) -> VCC
- D37 pad 4: Net-(D36-Pad2) -> Net-(D37-Pad4)
- D38 pad 2: Net-(D38-Pad2) -> Net-(D37-Pad4)
- D38 pad 3: Net-(C42-Pad1) -> VCC
- D38 pad 4: Net-(D37-Pad2) -> Net-(D38-Pad4)
- D39 pad 2: Net-(D39-Pad2) -> Net-(D38-Pad4)
- D39 pad 3: Net-(C41-Pad1) -> VCC
- D39 pad 4: Net-(D38-Pad2) -> Net-(D39-Pad4)
- D4 pad 3: Net-(C13-Pad1) -> VCC
- D40 pad 2: Net-(D30-Pad4) -> Net-(D39-Pad4)
- D40 pad 3: Net-(C40-Pad1) -> VCC
- D40 pad 4: Net-(D39-Pad2) -> unconnected-(D40-Pad4)
- D5 pad 3: Net-(C14-Pad1) -> VCC
- D6 pad 3: Net-(C15-Pad1) -> VCC
- D7 pad 3: Net-(C16-Pad1) -> VCC
- D8 pad 3: Net-(C17-Pad1) -> VCC
- D9 pad 3: Net-(C18-Pad1) -> VCC
- U1 pad 13: BUZZER -> BTN_DWN
- U1 pad 17: unconnected-(U1-Pad17) -> MOSI
- U1 pad 18: unconnected-(U1-Pad18) -> MISO
- U1 pad 23: unconnected-(U1-Pad23) -> TRIG
- U1 pad 24: unconnected-(U1-Pad24) -> ECHO
- U1 pad 5: BTN_DWN -> BUZZER
- U3 pad 10: NEO -> unconnected-(U3-Pad10)
Other:
- board size 118 x 118 mm -> 140 x 90 mm

Commit message: update
Parts:
- R15: moved to B.Cu
- moved R13 214.9 mm to (114.3, 94.0)
- moved D20 210.5 mm to (190.5, 58.4), turned to 180 degrees
- moved D19 201.2 mm to (213.4, 68.6), turned to 90 degrees
- moved D30 198.9 mm to (114.3, 58.4), turned to 180 degrees
- moved D29 188.2 mm to (121.9, 58.4), turned to 180 degrees
- moved D18 185.6 mm to (213.4, 76.2), turned to 90 degrees
- moved D28 177.8 mm to (129.5, 58.4), turned to 180 degrees
- moved C10 171.7 mm to (94.0, 134.6), turned to 180 degrees
- moved D17 171.3 mm to (213.4, 83.8), turned to 90 degrees
- moved R4 171.3 mm to (106.7, 81.3)
- moved D27 167.7 mm to (137.2, 58.4), turned to 180 degrees
- moved R5 164.0 mm to (171.9, 111.8)
- moved C6 162.3 mm to (198.1, 121.9)
- moved D50 160.9 mm to (185.4, 116.8)
- moved D26 158.0 mm to (144.8, 58.4), turned to 180 degrees
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
Commit message: update
Parts:
- moved R4 8.03 mm to (109.2, 73.7)
- moved R1 7.18 mm to (189.7, 116.8)
- moved C6 7.18 mm to (203.2, 116.8)
- moved R3 5.68 mm to (114.3, 73.7)
- moved C3 3.59 mm to (119.4, 73.7)
- moved C11 2.54 mm to (203.2, 134.6)
Changed lines of the file:
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@@
   )
   (footprint "footprints:C_0805_2012Metric" (layer "F.Cu")
-    (at 198.12 121.92)
+    (at 203.2 116.84)
     (descr "Capacitor SMD 0805 (2012 Metric), square (rectangular) end terminal, IPC_7351 nominal, (Body size source: http://www.tortai-tech.com/upload/download/2011102023233369053.pdf), generated with kicad-footprint-generator")
     (tags "capacitor")
@@
   )
   (footprint "footprints:C_0805_2012Metric" (layer "F.Cu")
-    (at 116.84 76.2)
+    (at 119.38 73.66)
     (descr "Capacitor SMD 0805 (2012 Metric), square (rectangular) end terminal, IPC_7351 nominal, (Body size source: http://www.tortai-tech.com/upload/download/2011102023233369053.pdf), generated with kicad-footprint-generator")
     (tags "capacitor")
@@
   )
   (footprint "footprints:R_0805_2012Metric" (layer "F.Cu")
-    (at 106.68 81.28)
+    (at 109.22 73.66)
     (descr "Resistor SMD 0805 (2012 Metric), square (rectangular) end terminal, IPC_7351 nominal, (Body size source: http://www.tortai-tech.com/upload/download/2011102023233369053.pdf), generated with kicad-footprint-generator")
     (tags "resistor")
@@
   )
   (footprint "footprints:C_0805_2012Metric" (layer "F.Cu")
-    (at 205.74 134.62)
+    (at 203.2 134.62)
     (descr "Capacitor SMD 0805 (2012 Metric), square (rectangular) end terminal, IPC_7351 nominal, (Body size source: http://www.tortai-tech.com/upload/download/2011102023233369053.pdf), generated with kicad-footprint-generator")
     (tags "capacitor")
@@
   )
   (footprint "footprints:R_0805_2012Metric" (layer "F.Cu")
-    (at 111.76 78.74)
+    (at 114.3 73.66)
     (descr "Resistor SMD 0805 (2012 Metric), square (rectangular) end terminal, IPC_7351 nominal, (Body size source: http://www.tortai-tech.com/upload/download/2011102023233369053.pdf), generated with kicad-footprint-generator")
     (tags "resistor")
@@
   )
   (footprint "footprints:R_0805_2012Metric" (layer "F.Cu")
-    (at 184.57 121.92)
+    (at 189.65 116.84)
     (descr "Resistor SMD 0805 (2012 Metric), square (rectangular) end terminal, IPC_7351 nominal, (Body size source: http://www.tortai-tech.com/upload/download/2011102023233369053.pdf), generated with kicad-footprint-generator")
     (tags "resistor")

Commit message: pcb-changes
Parts:
- J1: value PJ-102AH -> VAL**
- moved U3 32.1 mm to (135.9, 118.1), turned to 90 degrees
- moved U1 25.7 mm to (198.1, 76.2), turned to 0 degrees
- moved J2 16.8 mm to (111.8, 85.1), turned to 180 degrees
- moved R4 13.8 mm to (118.5, 83.8)
- moved R14 13.0 mm to (203.2, 68.6), turned to 180 degrees
- moved R2 13.0 mm to (190.5, 66.0), turned to 180 degrees
- moved C1 9.16 mm to (182.9, 81.3)
- moved Y1 9.16 mm to (185.4, 99.1)
- moved C2 9.16 mm to (188.0, 81.3)
- moved C6 9.16 mm to (198.1, 124.5), turned to 90 degrees
- moved R1 9.12 mm to (185.4, 124.9)
- moved D50 9.12 mm to (181.2, 124.9)
- moved U2 9.12 mm to (182.9, 114.3)
- moved C7 9.12 mm to (190.5, 114.7)
- moved C4 8.03 mm to (182.9, 86.4)
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Routing:
- net Net-(D4-Pad4): track 0.00 -> 13.8 mm
- net Net-(D2-Pad4): track 0.00 -> 13.8 mm
- net Net-(D10-Pad2): track 0.00 -> 13.8 mm
- net Net-(D8-Pad4): track 0.00 -> 13.8 mm
- net Net-(D10-Pad4): track 0.00 -> 13.8 mm
- net Net-(D7-Pad4): track 0.00 -> 13.8 mm
- net Net-(D3-Pad4): track 0.00 -> 13.8 mm
- net Net-(D1-Pad4): track 0.00 -> 13.8 mm
- net Net-(D6-Pad4): track 0.00 -> 13.8 mm
- net Net-(D5-Pad4): track 0.00 -> 13.8 mm
- net Net-(D11-Pad4): track 0.00 -> 13.8 mm

Commit message: PCB update
Parts:
- removed the H1 at (84.9, 56.2)
- removed the H2 at (214.9, 56.2)
- removed the H3 at (84.9, 136.2)
- removed the H4 at (214.9, 136.2)
- R15: moved to F.Cu
- moved R11 26.9 mm to (156.5, 129.0)
- moved SW3 26.4 mm to (155.9, 124.4)
- moved R10 23.3 mm to (144.3, 129.0), turned to 180 degrees
- moved SW2 23.3 mm to (144.3, 124.4)
- moved C6 22.9 mm to (177.8, 113.9)
- moved R5 20.4 mm to (150.0, 107.7)
- moved R14 16.3 mm to (190.5, 78.7), turned to 0 degrees
- moved C1 13.0 mm to (194.1, 87.9), turned to 90 degrees
- moved R12 12.4 mm to (167.3, 129.0), turned to 180 degrees
- moved SW4 12.1 mm to (167.1, 124.4)
- moved C5 10.8 mm to (180.8, 94.5)
- moved R9 9.65 mm to (132.6, 129.5), turned to 180 degrees
- moved C4 9.58 mm to (188.0, 94.5)
- moved SW1 9.14 mm to (133.1, 124.4)
- moved R2 7.62 mm to (190.5, 73.7)
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Routing:
- net GND: track 0.00 -> 565.4 mm, vias 0 -> 16
- net VCC: track 0.00 -> 557.9 mm, vias 0 -> 12
- net RESET: track 0.00 -> 134.2 mm
- net SCL: track 0.00 -> 117.5 mm, vias 0 -> 3
- net NEO: track 0.00 -> 112.2 mm, vias 0 -> 2
- net SDA: track 0.00 -> 111.5 mm, vias 0 -> 4
- net BTN_ALARM: track 0.00 -> 102.3 mm
- net TRIG: track 0.00 -> 93.3 mm, vias 0 -> 3
- net ECHO: track 0.00 -> 89.2 mm, vias 0 -> 3
- net BUZZER: track 0.00 -> 86.4 mm
- net BTN_UP: track 0.00 -> 83.1 mm, vias 0 -> 3
- net RXD: track 0.00 -> 81.4 mm
- net TXD: track 0.00 -> 81.4 mm
- net LED_SCK: track 0.00 -> 79.5 mm, vias 0 -> 2
- net BTN_DWN: track 0.00 -> 79.0 mm, vias 0 -> 4
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- added copper zone on B.Cu, net GND
- added copper zone on F.Cu, net VCC

Commit message: update
Routing:
- net GND: track 565.4 -> 584.6 mm, vias 16 -> 18
- net VCC: track 557.9 -> 568.4 mm, vias 12 -> 14
Changed lines of the file:
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@@
   (segment (start 199.224311 85.557422) (end 198.577422 86.204311) (width 0.2032) (layer "F.Cu") (net 2))
   (segment (start 198.577422 86.204311) (end 196.7987 86.204311) (width 0.2032) (layer "F.Cu") (net 2))
+  (segment (start 194.564 109.22) (end 194.564 110.236) (width 0.2032) (layer "F.Cu") (net 2))
   (segment (start 142.33 56.806) (end 142.33 56.82) (width 0.2032) (layer "F.Cu") (net 2))
   (segment (start 202.633622 136.22) (end 204.05 134.803622) (width 0.2032) (layer "F.Cu") (net 2))
@@
   (segment (start 157.57 56.806) (end 157.57 56.82) (width 0.2032) (layer "F.Cu") (net 2))
   (segment (start 84.746 98.97) (end 84.76 98.97) (width 0.2032) (layer "F.Cu") (net 2))
+  (segment (start 194.32 97.8) (end 194.056 97.536) (width 0.2032) (layer "F.Cu") (net 2))
   (segment (start 151.892 128.016) (end 151.384 128.524) (width 0.2032) (layer "F.Cu") (net 2))
   (segment (start 111.76 85.344) (end 110.316 85.344) (width 0.2032) (layer "F.Cu") (net 2))
@@
   (segment (start 215.9 82.296) (end 214.974 81.37) (width 0.2032) (layer "F.Cu") (net 2))
   (segment (start 111.85 56.82) (end 111.045689 56.015689) (width 0.2032) (layer "F.Cu") (net 2))
+  (segment (start 198.12 97.8) (end 194.32 97.8) (width 0.2032) (layer "F.Cu") (net 2))
   (segment (start 150.876 55.88) (end 149.95 56.806) (width 0.2032) (layer "F.Cu") (net 2))
   (segment (start 172.81 56.806) (end 172.81 56.82) (width 0.2032) (layer "F.Cu") (net 2))
+  (segment (start 194.564 110.236) (end 193.04 111.76) (width 0.2032) (layer "F.Cu") (net 2))
   (segment (start 84.76 106.59) (end 84.418 106.59) (width 0.2032) (layer "F.Cu") (net 2))
   (segment (start 83.312 67.564) (end 84.328 68.58) (width 0.2032) (layer "F.Cu") (net 2))
@@
   (via (at 177.8 111.76) (size 0.8128) (drill 0.4064) (layers "F.Cu" "B.Cu") (net 2))
   (via (at 137.668 128.524) (size 0.8128) (drill 0.4064) (layers "F.Cu" "B.Cu") (net 2))
+  (via (at 194.564 109.22) (size 0.8128) (drill 0.4064) (layers "F.Cu" "B.Cu") (net 2))
   (via (at 162.56 128.524) (size 0.8128) (drill 0.4064) (layers "F.Cu" "B.Cu") (net 2))
   (via (at 196.088 86.915011) (size 0.8128) (drill 0.4064) (layers "F.Cu" "B.Cu") (net 2))
@@
   (via (at 128.524 128.524) (size 0.8128) (drill 0.4064) (layers "F.Cu" "B.Cu") (net 2))
   (via (at 160.528 128.524) (size 0.8128) (drill 0.4064) (layers "F.Cu" "B.Cu") (net 2))
+  (via (at 194.056 97.536) (size 0.8128) (drill 0.4064) (layers "F.Cu" "B.Cu") (net 2))
   (segment (start 185.42 74.168) (end 185.42 78.232) (width 0.2032) (layer "B.Cu") (net 2))
+  (segment (start 194.056 97.536) (end 194.056 108.712) (width 0.2032) (layer "B.Cu") (net 2))
+  (segment (start 194.056 108.712) (end 194.564 109.22) (width 0.2032) (layer "B.Cu") (net 2))
   (segment (start 115.648 93.98) (end 115.99 93.638) (width 0.2032) (layer "F.Cu") (net 3))
   (segment (start 106.68 93.98) (end 115.648 93.98) (width 0.2032) (layer "F.Cu") (net 3))
@@
   (segment (start 89.408 85.344) (end 88.302 86.45) (width 0.2032) (layer "F.Cu") (net 5))
   (segment (start 146.29 60.96) (end 140.208 60.96) (width 0.2032) (layer "F.Cu") (net 5))
+  (segment (start 185.4567 82.13) (end 186.436 83.1093) (width 0.2032) (layer "F.Cu") (net 5))
   (segment (start 118.665689 132.215689) (end 119.47 133.02) (width 0.2032) (layer "F.Cu") (net 5))
   (segment (start 158.496 129.032) (end 159.004 129.54) (width 0.2032) (layer "F.Cu") (net 5))
@@
   (segment (start 116.75 60.02) (end 115.81 60.96) (width 0.2032) (layer "F.Cu") (net 5))
   (segment (start 164.25 132.08) (end 165.19 133.02) (width 0.2032) (layer "F.Cu") (net 5))
+  (segment (start 191.15973 81.12827) (end 189.65 79.61854) (width 0.2032) (layer "F.Cu") (net 5))
   (segment (start 210.955689 85.465689) (end 210.955689 79.454311) (width 0.2032) (layer "F.Cu") (net 5))
   (segment (start 89.394 110.744) (end 89.408 110.744) (width 0.2032) (layer "F.Cu") (net 5))
@@
   (segment (start 134.71 133.02) (end 135.65 132.08) (width 0.2032) (layer "F.Cu") (net 5))
   (segment (start 120.41 132.08) (end 126.15 132.08) (width 0.2032) (layer "F.Cu") (net 5))
+  (segment (start 189.65 79.61854) (end 189.65 78.74) (width 0.2032) (layer "F.Cu") (net 5))
   (segment (start 125.31 60.96) (end 124.37 60.02) (width 0.2032) (layer "F.Cu") (net 5))
   (segment (start 161.53 60.96) (end 155.79 60.96) (width 0.2032) (layer "F.Cu") (net 5))
@@
   (segment (start 86.76592 64.78408) (end 86.76592 70.104) (width 0.2032) (layer "F.Cu") (net 5))
   (segment (start 88.302 109.31) (end 87.96 109.31) (width 0.2032) (layer "F.Cu") (net 5))
+  (segment (start 184.912 82.13) (end 185.4567 82.13) (width 0.2032) (layer "F.Cu") (net 5))
   (via (at 190.5 131.255011) (size 0.8128) (drill 0.4064) (layers "F.Cu" "B.Cu") (net 5))
   (via (at 133.604 131.255011) (size 0.8128) (drill 0.4064) (layers "F.Cu" "B.Cu") (net 5))
@@
   (via (at 199.644 105.156) (size 0.8128) (drill 0.4064) (layers "F.Cu" "B.Cu") (net 5))
   (via (at 135.128 129.833611) (size 0.8128) (drill 0.4064) (layers "F.Cu" "B.Cu") (net 5))
+  (via (at 191.15973 81.12827) (size 0.8128) (drill 0.4064) (layers "F.Cu" "B.Cu") (net 5))
   (via (at 207.674325 106.582325) (size 0.8128) (drill 0.4064) (layers "F.Cu" "B.Cu") (net 5))
+  (via (at 186.436 83.1093) (size 0.8128) (drill 0.4064) (layers "F.Cu" "B.Cu") (net 5))
   (via (at 146.812 129.54) (size 0.8128) (drill 0.4064) (layers "F.Cu" "B.Cu") (net 5))
   (segment (start 199.644 105.156) (end 203.708 109.22) (width 0.2032) (layer "B.Cu") (net 5))
@@
   (segment (start 204.299528 107.52461) (end 205.241813 106.582325) (width 0.2032) (layer "B.Cu") (net 5))
   (segment (start 190.5 131.255011) (end 190.5 123.952) (width 0.2032) (layer "B.Cu") (net 5))
+  (segment (start 188.41703 81.12827) (end 191.15973 81.12827) (width 0.2032) (layer "B.Cu") (net 5))
+  (segment (start 186.436 83.1093) (end 188.41703 81.12827) (width 0.2032) (layer "B.Cu") (net 5))
   (segment (start 146.812 129.54) (end 145.096989 131.255011) (width 0.2032) (layer "B.Cu") (net 5))
   (segment (start 133.7066 131.255011) (end 133.604 131.255011) (width 0.2032) (layer "B.Cu") (net 5))

Commit message: pcb
Parts:
- C7: value 0.1uf -> C_0805_1uf
- J1: value VAL** -> Power_inlet_vertical; footprint footprints:PJ-102AH -> footprints:Wurth-694106402002; moved to B.Cu
- moved J1 35.6 mm to (172.5, 112.3), turned to 90 degrees
- moved C2 20.1 mm to (176.8, 99.7)
- moved C1 15.5 mm to (179.6, 82.3), turned to 0 degrees
- moved BZ1 3.30 mm to (110.0, 94.0)
- moved C4 1.63 mm to (189.0, 95.8)
- moved C5 1.30 mm to (180.6, 95.8)
- moved C3 1.02 mm to (118.9, 71.6)
- moved R4 1.02 mm to (118.9, 78.7)
- moved R10 0.44 mm to (144.8, 129.0)
- moved R9 0.34 mm to (132.9, 129.5)
Connections:
- D10 pad 3: VCC -> unconnected-(D10-Pad3)
- U1 pad 22: unconnected-(U1-Pad22) -> GND
Routing:
- net GND: track 584.6 -> 177.0 mm, vias 18 -> 59
- net VCC: track 568.4 -> 355.8 mm, vias 14 -> 49
- net TRIG: track 93.3 -> 0.00 mm, vias 3 -> 0
- net ECHO: track 89.2 -> 0.00 mm, vias 3 -> 0
- net BTN_ALARM: track 102.3 -> 16.7 mm
- net RXD: track 81.4 -> 0.00 mm
- net TXD: track 81.4 -> 0.00 mm
- net LED_SCK: track 79.5 -> 0.00 mm, vias 2 -> 0
- net BTN_UP: track 83.1 -> 16.5 mm, vias 3 -> 0
- net BTN_DWN: track 79.0 -> 16.4 mm, vias 4 -> 0
- net Net-(C1-Pad1): track 47.6 -> 0.00 mm, vias 2 -> 0
- net BTN_PAUSE: track 63.1 -> 17.7 mm, vias 2 -> 0
- net DISP_CLK: track 43.0 -> 86.6 mm
- net MOSI: track 42.7 -> 0.00 mm, vias 1 -> 0
- net DISP_LOAD: track 36.4 -> 0.00 mm
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- added copper zone on F.Cu, net GND
- removed copper zone on F.Cu, net VCC

Commit message: update
Parts:
- moved C1 32.8 mm to (209.0, 96.6), turned to 90 degrees
- moved D50 25.6 mm to (206.8, 127.8), turned to 90 degrees
- moved R1 21.6 mm to (206.8, 123.6), turned to 90 degrees
- moved C2 19.3 mm to (195.6, 95.2)
Routing:
- net VCC: track 355.8 -> 451.9 mm, vias 49 -> 41
- net BTN_ALARM: track 16.7 -> 108.2 mm, vias 0 -> 2
- net TXD: track 0.00 -> 81.6 mm, vias 0 -> 1
- net RXD: track 0.00 -> 81.4 mm, vias 0 -> 1
- net TRIG: track 0.00 -> 66.9 mm
- net ECHO: track 0.00 -> 63.0 mm, vias 0 -> 1
- net LED_SCK: track 0.00 -> 62.3 mm, vias 0 -> 1
- net BTN_UP: track 16.5 -> 78.1 mm, vias 0 -> 3
- net MOSI: track 0.00 -> 47.4 mm, vias 0 -> 3
- net BTN_PAUSE: track 17.7 -> 63.0 mm
- net DISP_LOAD: track 0.00 -> 40.3 mm, vias 0 -> 1
- net DISP_CLK: track 86.6 -> 49.6 mm
- net /DIG_2: track 0.00 -> 36.6 mm, vias 0 -> 2
- net Net-(D31-Pad4): track 0.00 -> 26.0 mm
- net RESET: track 114.0 -> 123.8 mm, vias 1 -> 3
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