File: clock/clock.kicad_pcb (KiCad board)
At the start: 2 copper layers, 140 x 90 mm, 88 parts, among them J1 Power_inlet_vertical, J2 Conn_01x06, J3 Conn_02x03_Odd_Even, SW1 Omron_B3F_SPST, SW2 Omron_B3F_SPST, SW3 Omron_B3F_SPST, SW4 Omron_B3F_SPST, SW5 Omron_B3F_SPST, U1 ATmega328-PU, U2 L7805, U3 MAX7219, U4 DS1307_DIP-8, U5 UltrasonicModule, Y1 16MHz, Y2 Crystal_32768Hz

Commit message: update
Routing:
- net GND: track 183.1 -> 289.1 mm, vias 58 -> 68
- net BTN_DWN: track 16.4 -> 75.0 mm, vias 0 -> 3
- net /SEG_C: track 18.4 -> 8.12 mm
- net /SEG_B: track 25.0 -> 27.7 mm, vias 2 -> 3
- net DISP_LOAD: track 40.3 -> 38.0 mm
- net VCC: track 451.9 -> 453.8 mm, vias 41 -> 42
- net MOSI: track 47.4 -> 48.9 mm
- net /SEG_G: track 9.61 -> 8.37 mm
- net /DIG_2: track 36.6 -> 37.5 mm
- net /DIG_3: track 16.3 -> 15.5 mm
- net /DIG_4: track 30.4 -> 29.7 mm, vias 1 -> 2
- net BTN_ALARM: vias 2 -> 4
- added copper zone on F.Cu, net VCC
- removed copper zone on F.Cu, net GND

Commit message: update
Connections:
- DS1 pad 10: /DIG_2 -> GND
- DS1 pad 6: /DIG_3 -> GND
- U3 pad 5: unconnected-(U3-Pad5) -> GND
- U3 pad 6: /DIG_2 -> GND
- U3 pad 7: /DIG_3 -> GND
- U3 pad 8: unconnected-(U3-Pad8) -> GND
Routing:
- net /DIG_2: track 37.5 -> 0.00 mm, vias 2 -> 0
- net GND: track 289.1 -> 309.2 mm, vias 68 -> 69
- net /DIG_3: track 15.5 -> 0.00 mm
- net MOSI: track 48.9 -> 47.4 mm
Other:
- board text added: "TICK TOCK"
